Commit message: add aruco detection

File: src/ur_robotiq_gazebo/urdf/ur.xacro (robot description, xacro)
@@ -57,5 +57,5 @@
   <xacro:include filename="$(find ur_robotiq_gazebo)/urdf/_d435.urdf.xacro" />
   <xacro:sensor_d435 parent="wrist_3_link" name="camera_depth" topics_ns="camera_depth">
-    <origin xyz="0.033891980 0 0.018843205478" rpy="0 ${-pi/2} 0"/>
+    <origin xyz="0.08 0 0.05" rpy="0 ${-pi/2} 0"/>
   </xacro:sensor_d435>
   <!--
